File: PCB/KiCad Files/Wireless_Communication_Board(WCB)V2.1/Wireless_Communication_Board(WCB)V2.kicad_pcb (KiCad board)
At the start: 4 copper layers, 52.5 x 38.3 mm, 44 parts, among them J1 USB_B_Micro, J2 Power In, J3 Conn_01x04, J4 Conn_01x04, J5 Conn_01x04, J6 Conn_01x04, J7 Conn_01x04, Q2 UMH3N, U1 ESP32-PICO-MINI-02, U2 CP2102N-A02-GQFN28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

Commit message: Updated the Readme and removed old images.
Other:
- board text added: "3.2mm Diameter"
- board text added: "31mm"
- board text added: "38.35mm"
- board text added: "45.5mm"
- board text added: "52.5mm"
Changed lines of the file:
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@@
   (gr_rect (start 123.19 110.49) (end 127 113.03) (layer "F.CrtYd") (width 0.05) (fill none))
   (gr_rect (start 123.464 99.752) (end 112.776 89.662) (layer "F.CrtYd") (width 0.05) (fill none))
+  (gr_line (start 99.39 126.238) (end 105.334 126.238) (layer "User.1") (width 0.2))
+  (gr_line (start 140.081 129.286) (end 158.115 129.286) (layer "User.1") (width 0.2))
+  (gr_line (start 157.988 131.826) (end 157.988 126.39) (layer "User.1") (width 0.2))
+  (gr_line (start 161.27 122.682) (end 161.27 110.998) (layer "User.1") (width 0.2))
+  (gr_line (start 102.362 87.884) (end 102.362 101.6) (layer "User.1") (width 0.2))
+  (gr_line (start 102.362 112.522) (end 102.362 126.238) (layer "User.1") (width 0.2))
+  (gr_line (start 158.056 91.754) (end 164 91.754) (layer "User.1") (width 0.2))
+  (gr_line (start 109 87.436) (end 109 82) (layer "User.1") (width 0.2))
+  (gr_line (start 105.41 131.826) (end 105.41 126.39) (layer "User.1") (width 0.2))
+  (gr_line (start 136.398 84.492) (end 154.432 84.492) (layer "User.1") (width 0.2))
+  (gr_line (start 154.5 87.436) (end 154.5 82) (layer "User.1") (width 0.2))
+  (gr_line (start 161.27 91.694) (end 161.27 105.41) (layer "User.1") (width 0.2))
+  (gr_line (start 99.39 87.884) (end 105.334 87.884) (layer "User.1") (width 0.2))
+  (gr_line (start 154.5 91.5) (end 156.718 87.376) (layer "User.1") (width 0.2))
+  (gr_line (start 105.537 129.286) (end 122.047 129.286) (layer "User.1") (width 0.2))
+  (gr_line (start 158.056 122.754) (end 164 122.754) (layer "User.1") (width 0.2))
+  (gr_line (start 108.966 84.492) (end 125.476 84.492) (layer "User.1") (width 0.2))
   (gr_text "5V" (at 148.082 108.966) (layer "F.SilkS")
     (effects (font (size 0.8 0.8) (thickness 0.15)))
@@
     (effects (font (size 0.8 0.8) (thickness 0.15)))
   )
+  (gr_text "31mm" (at 161.798 107.696) (layer "User.1")
+    (effects (font (size 1.5 1.5) (thickness 0.3)))
+  )
+  (gr_text "45.5mm" (at 130.81 84.582) (layer "User.1")
+    (effects (font (size 1.5 1.5) (thickness 0.3)))
+  )
+  (gr_text "38.35mm" (at 100.584 107.188) (layer "User.1")
+    (effects (font (size 1.5 1.5) (thickness 0.3)))
+  )
+  (gr_text "52.5mm" (at 131.826 129.54) (layer "User.1")
+    (effects (font (size 1.5 1.5) (thickness 0.3)))
+  )
+  (gr_text "3.2mm\nDiameter" (at 160.528 85.09) (layer "User.1")
+    (effects (font (size 1.5 1.5) (thickness 0.3)))
+  )
   (segment (start 128.218 115.01) (end 127.718 114.51) (width 0.25) (layer "F.Cu") (net 1))
