File: PCB/KiCad Files/Wireless_Communication_Board(WCB)_V1.0/Wireless_Communication_Board(WCB)_V1.kicad_pcb (KiCad board)
At the start: 2 copper layers, 54.8 x 53 mm, 14 parts, among them J1 S1, J2 S2, J3 S3, J4 S4, J5 S5, J6 Screw_Terminal_01x02, U1 LilyGo_TTGO_T7_V1.5

Commit message: Updated the Readme and removed old images.
Other:
- board text added: "3.2mm Diameter"
- board text added: "45.5mm"
- board text added: "47.5mm"
- board text added: "53mm"
- board text added: "54.75mm"
Changed lines of the file:
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@@
   (gr_line (start 114 120) (end 114 67) (layer "Edge.Cuts") (width 0.1))
   (gr_line (start 168.762 120) (end 114 120) (layer "Edge.Cuts") (width 0.1))
+  (gr_line (start 145.288 64.516) (end 165.1 64.516) (layer "User.1") (width 0.15))
+  (gr_line (start 173.944 70.612) (end 168.944 70.612) (layer "User.1") (width 0.15))
+  (gr_line (start 168.656 120) (end 168.656 125) (layer "User.1") (width 0.15))
+  (gr_line (start 146.558 122.682) (end 168.656 122.682) (layer "User.1") (width 0.15))
+  (gr_line (start 114 119.888) (end 109 119.888) (layer "User.1") (width 0.15))
+  (gr_line (start 114.046 122.5) (end 136.906 122.682) (layer "User.1") (width 0.15))
+  (gr_line (start 114 67.056) (end 109 67.056) (layer "User.1") (width 0.15))
+  (gr_line (start 173.944 116.332) (end 168.944 116.332) (layer "User.1") (width 0.15))
+  (gr_line (start 114.046 120) (end 114.046 125) (layer "User.1") (width 0.15))
+  (gr_line (start 165.1 62.016) (end 165.1 67.016) (layer "User.1") (width 0.15))
+  (gr_line (start 111.5 67.056) (end 111.252 89.154) (layer "User.1") (width 0.15))
+  (gr_line (start 117.856 64.516) (end 137.414 64.516) (layer "User.1") (width 0.15))
+  (gr_line (start 111.5 119.888) (end 111.506 93.726) (layer "User.1") (width 0.15))
+  (gr_line (start 171.444 116.332) (end 171.45 94.488) (layer "User.1") (width 0.15))
+  (gr_line (start 171.444 70.612) (end 171.45 89.916) (layer "User.1") (width 0.15))
+  (gr_line (start 117.856 62.016) (end 117.856 67.016) (layer "User.1") (width 0.15))
+  (gr_line (start 165.1 70.612) (end 167.386 65.786) (layer "User.1") (width 0.15))
   (gr_text "TD0/1	TD0/SD1" (at 141.743905 100.584) (layer "F.SilkS")
     (effects (font (size 0.25 0.25) (thickness 0.0625)))
@@
     (effects (font (size 0.5 0.5) (thickness 0.125)))
   )
+  (gr_text "47.5mm" (at 141.478 64.698) (layer "User.1")
+    (effects (font (size 1 1) (thickness 0.15)))
+  )
+  (gr_text "3.2mm\nDiameter" (at 170.688 64.262) (layer "User.1")
+    (effects (font (size 1 1) (thickness 0.15)))
+  )
+  (gr_text "45.5mm" (at 172.212 92.456) (layer "User.1")
+    (effects (font (size 1 1) (thickness 0.15)))
+  )
+  (gr_text "53mm" (at 110.236 91.44) (layer "User.1")
+    (effects (font (size 1 1) (thickness 0.15)))
+  )
+  (gr_text "54.75mm" (at 141.732 122.682) (layer "User.1")
+    (effects (font (size 1 1) (thickness 0.15)))
+  )
   (segment (start 156.034 83.47) (end 154.859489 82.295489) (width 0.25) (layer "B.Cu") (net 3))
