File: PCB/KiCad Files/Wireless_Communincation_Board(WCB)V2.3/Wireless_Communincation_Board(WCB)V2.kicad_pcb (KiCad board)
At the start: 4 copper layers, 70.2 x 70.1 mm, 65 parts, among them J1 USB_B_Micro, J2 Power In, J3 Conn_01x04, J4 Conn_01x04, J5 Conn_01x04, J6 Conn_01x04, J7 Conn_01x04, J8 Conn_01x01, Q2 UMH3N, U1 ESP32-PICO-MINI-02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

Commit message: Working on updated to improve functionality
Parts:
- moved G*** 1.05 mm to (131.1, 109.2)
Changed lines of the file:
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@@
   )
   (footprint "Logos:r2logoLarge" (layer "B.Cu")
-    (at 130.048 108.966 180)
+    (at 131.064 109.22 180)
     (attr board_only exclude_from_pos_files exclude_from_bom)
     (fp_text reference "G***" (at -0.762 -2.286) (layer "B.SilkS") hide
@@
   (gr_line (start 170.668 91.948) (end 170.668 105.664) (layer "User.1") (width 0.2))
   (gr_line (start 89.992 87.884) (end 95.936 87.884) (layer "User.1") (width 0.2))
-  (gr_line (start 154.686 91.44) (end 160.528 80.01) (layer "User.1") (width 0.2))
+  (gr_line (start 154.686 91.44) (end 168.91 81.534) (layer "User.1") (width 0.2))
   (gr_line (start 105.537 135.382) (end 122.047 135.382) (layer "User.1") (width 0.2))
   (gr_line (start 167.454 123.008) (end 173.398 123.008) (layer "User.1") (width 0.2))
@@
     (effects (font (size 1.5 1.5) (thickness 0.3)))
   )
-  (gr_text "3.2mm\nDiameter" (at 164.084 77.216) (layer "User.1")
-    (effects (font (size 1.5 1.5) (thickness 0.3)))
-  )
+  (gr_text "3.2mm\nDiameter" (at 172.212 78.486) (layer "User.1")
+    (effects (font (size 1.5 1.5) (thickness 0.3)))
+  )
