File: PCB/KiCad Files/Wireless_Communincation_Board(WCB)V2.3/Wireless_Communincation_Board(WCB)V2.kicad_sch (KiCad schematic)
At the start: 37 parts, among them J1 USB_B_Micro, J2 Power In, J3 Conn_01x04, J4 Conn_01x04, J5 Conn_01x04, J6 Conn_01x04, J7 Conn_01x04, J8 Conn_01x01, Q2 UMH3N, U1 ESP32-PICO-MINI-02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

Commit message: updated the pcb
Parts:
- D1: footprint Custom:SOD3716X135N -> 01-Custom:SOD3716X135N
- L2: footprint Custom:WS2812B-2020 -> 01-Custom:WS2812B-2020
- Q2: footprint Custom:SOT65P230X110-6N -> 01-Custom:SOT65P230X110-6N
- S1: footprint Custom:SW_TL3342F160QG -> 01-Custom:SW_TL3342F160QG
- U1: footprint Custom:MODULE_ESP32-PICO-MINI-02 -> 01-Custom:MODULE_ESP32-PICO-MINI-02
