File: PCB/KiCad Files/Wireless_Communincation_Board(WCB)V2.3/Wireless_Communincation_Board(WCB)V2-backups/Wireless_Communincation_Board(WCB)V2-2024-04-12_113054 2/Wireless_Communincation_Board(WCB)V2.kicad_pcb (KiCad board)
At the start: 4 copper layers, 70.2 x 70.1 mm, 65 parts, among them J1 USB_B_Micro, J2 Power In, J3 Conn_01x04, J4 Conn_01x04, J5 Conn_01x04, J6 Conn_01x04, J7 Conn_01x04, J8 Conn_01x01, Q2 UMH3N, U1 ESP32-PICO-MINI-02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

Commit message: updated the pcb
Parts:
- D1: footprint 01-Custom:SOD3716X135N -> Custom:SOD3716X135N
- L2: footprint 01-Custom:WS2812B-2020 -> Custom:WS2812B-2020
- Q2: footprint 01-Custom:SOT65P230X110-6N -> Custom:SOT65P230X110-6N
- S1: footprint 01-Custom:SW_TL3342F160QG -> Custom:SW_TL3342F160QG
- U1: footprint 01-Custom:MODULE_ESP32-PICO-MINI-02 -> Custom:MODULE_ESP32-PICO-MINI-02
Routing:
- net +3V3: track 9.86 -> 4.85 mm
- net +5V: track 23.1 -> 18.9 mm
- net GND: track 124.8 -> 121.9 mm
