File: PCB/KiCad Files/Wireless Communication Board (WCB)V2.4/Wireless_Communication_Board(WCB)V2_4.kicad_pro/Wireless_Communication_Board(WCB)V2_4.kicad_pro.kicad_sch (KiCad schematic)
At the start: 37 parts, among them J1 USB_B_Micro, J2 Power In, J3 Conn_01x04, J4 Conn_01x04, J5 Conn_01x04, J6 Conn_01x04, J7 Conn_01x04, J8 Conn_01x01, Q2 UMH3N, U1 ESP32-PICO-MINI-02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

Commit message: updated part in the schematic due to obsolete regulator
Parts:
- U3: LCSC C2876187 -> C575581
