File: PCB/Wireless Communication Board (WCB)V3.1/Wireless Communication Board (WCB)V3.1.kicad_pcb (KiCad board)
At the start: 2 copper layers, 57.5 x 71.5 mm, 14 parts, among them J1 Serial 1, J2 Serial 2, J3 Serial 3, J4 Serial 4, J5 Serial 5, J6 Power, U1 ESP32-S3-DEVKITC-1-N8R2

Commit message: Changed the code to recognize version 31 instead of 30
Updated the readme as well.
Other:
- board text added: "3.2mm diameter"
- board text added: "50.5mm"
- board text added: "57.5mm"
- board text added: "64.5mm"
- board text added: "71.5mm"
